File: minimal-atmega328p.kicad_pcb (KiCad board)
At the start: 2 copper layers, 9 parts, among them J1 Conn_01x14_Male, J2 Conn_01x06_Male, J3 Conn_01x14_Male, U1 ATmega328P-PU, Y1 16MHz

Commit message: add diode
Parts:
- added D1: DIODE, Diode_THT:D_A-405_P2.54mm_Vertical_AnodeUp, F.Cu at (165.1, 85.2)
- moved C3 2.54 mm to (165.1, 93.3)
- moved R1 2.00 mm to (165.2, 98.6)
- moved J2 0.73 mm to (169.3, 86.0)
Routing:
- net Net-(C3-Pad1): track 9.55 -> 3.67 mm
- net /DTR: track 9.80 -> 7.16 mm
- net /TXD: track 12.9 -> 12.1 mm
- net /RXD: track 16.5 -> 15.7 mm
Changed lines of the file:
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@@
     (thickness 1.6)
     (drawings 0)
-    (tracks 78)
+    (tracks 74)
     (zones 0)
-    (modules 9)
+    (modules 10)
     (nets 27)
   )
@@
     (add_net "Net-(C2-Pad1)")
     (add_net "Net-(C3-Pad1)")
+    (add_net "Net-(J1-Pad1)")
+    (add_net "Net-(J1-Pad10)")
+    (add_net "Net-(J1-Pad2)")
+    (add_net "Net-(J1-Pad3)")
+    (add_net "Net-(J1-Pad9)")
+    (add_net "Net-(J2-Pad6)")
+    (add_net "Net-(J3-Pad8)")
+    (add_net "Net-(U1-Pad21)")
+  )
+  (module Diode_THT:D_A-405_P2.54mm_Vertical_AnodeUp (layer F.Cu)
+    (at 165.06952 85.15858 270)
+    (descr "Diode, A-405 series, Axial, Vertical, pin pitch=2.54mm, , length*diameter=5.2*2.7mm^2, , http://www.diodes.com/_files/packages/A-405.pdf")
+    (tags "Diode A-405 series Axial Vertical pin pitch 2.54mm  length 5.2mm diameter 2.7mm")
+    (fp_text reference D1 (at 1.27 -2.47 90) (layer F.SilkS)
+      (effects (font (size 1 1) (thickness 0.15)))
+    )
+    (fp_text value DIODE (at 1.27 3.359 90) (layer F.Fab)
+      (effects (font (size 1 1) (thickness 0.15)))
+    )
+    (fp_text user A (at 4.44 0 90) (layer F.SilkS)
+      (effects (font (size 1 1) (thickness 0.15)))
+    )
+    (fp_text user A (at 4.44 0 90) (layer F.Fab)
+      (effects (font (size 1 1) (thickness 0.15)))
+    )
+    (fp_text user %R (at 1.27 -2.47 90) (layer F.Fab)
+      (effects (font (size 1 1) (thickness 0.15)))
+    )
+    (fp_line (start 3.69 -1.6) (end -1.6 -1.6) (layer F.CrtYd) (width 0.05))
+    (fp_line (start 3.69 1.6) (end 3.69 -1.6) (layer F.CrtYd) (width 0.05))
+    (fp_line (start -1.6 1.6) (end 3.69 1.6) (layer F.CrtYd) (width 0.05))
+    (fp_line (start -1.6 -1.6) (end -1.6 1.6) (layer F.CrtYd) (width 0.05))
+    (fp_line (start 0 0) (end 2.54 0) (layer F.Fab) (width 0.1))
+    (fp_circle (center 0 0) (end 1.35 0) (layer F.Fab) (width 0.1))
+    (fp_arc (start 0 0) (end 1.113239 -0.9) (angle -278.451986) (layer F.SilkS) (width 0.12))
+    (pad 2 thru_hole oval (at 2.54 0 270) (size 1.8 1.8) (drill 0.9) (layers *.Cu *.Mask)
+      (net 9 +5V))
+    (pad 1 thru_hole rect (at 0 0 270) (size 1.8 1.8) (drill 0.9) (layers *.Cu *.Mask)
+      (net 4 "Net-(C3-Pad1)"))
+    (model ${KISYS3DMOD}/Diode_THT.3dshapes/D_A-405_P2.54mm_Vertical_AnodeUp.wrl
+      (at (xyz 0 0 0))
+      (scale (xyz 1 1 1))
+      (rotate (xyz 0 0 0))
+    )
   )
   (module Capacitor_THT:C_Disc_D3.8mm_W2.6mm_P2.50mm (layer B.Cu)
@@
   )
   (module Capacitor_THT:C_Disc_D3.8mm_W2.6mm_P2.50mm (layer F.Cu)
-    (at 165.69182 90.79738 90)
+    (at 165.10762 93.27134 90)
     (descr "C, Disc series, Radial, pin pitch=2.50mm, , diameter*width=3.8*2.6mm^2, Capacitor, http://www.vishay.com/docs/45233/krseries.pdf")
     (tags "C Disc series Radial pin pitch 2.50mm  diameter 3.8mm width 2.6mm Capacitor")
@@
   )
   (module Connector_PinHeader_2.54mm:PinHeader_1x06_P2.54mm_Vertical (layer F.Cu)
-    (at 169.99712 86.15426)
+    (at 169.27576 86.0425)
     (descr "Through hole straight pin header, 1x06, 2.54mm pitch, single row")
     (tags "Through hole pin header THT 1x06 2.54mm single row")
@@
   )
   (module Resistor_THT:R_Axial_DIN0207_L6.3mm_D2.5mm_P2.54mm_Vertical (layer F.Cu)
-    (at 165.6969 96.67494 90)
+    (at 165.1508 98.60026 90)
     (descr "Resistor, Axial_DIN0207 series, Axial, Vertical, pin pitch=2.54mm, 0.25W = 1/4W, length*diameter=6.3*2.5mm^2, http://cdn-reichelt.de/documents/datenblatt/B400/1_4W%23YAG.pdf")
     (tags "Resistor Axial_DIN0207 series Axial Vertical pin pitch 2.54mm 0.25W = 1/4W length 6.3mm diameter 2.5mm")
@@
   (segment (start 136.92566 91.96578) (end 131.57454 91.96578) (width 0.25) (layer B.Cu) (net 3))
   (segment (start 161.15538 87.90686) (end 160.91916 88.14308) (width 0.25) (layer F.Cu) (net 4))
-  (segment (start 163.03752 88.14308) (end 160.91916 88.14308) (width 0.25) (layer F.Cu) (net 4))
-  (segment (start 165.69182 90.79738) (end 163.03752 88.14308) (width 0.25) (layer F.Cu) (net 4))
-  (segment (start 165.69182 94.12986) (end 165.6969 94.13494) (width 0.25) (layer F.Cu) (net 4))
-  (segment (start 165.69182 90.79738) (end 165.69182 94.12986) (width 0.25) (layer F.Cu) (net 4))
-  (segment (start 169.99712 96.31426) (end 167.65016 93.9673) (width 0.25) (layer F.Cu) (net 5))
-  (segment (start 167.65016 90.25572) (end 165.69182 88.29738) (width 0.25) (layer F.Cu) (net 5))
-  (segment (start 167.65016 93.9673) (end 167.65016 90.25572) (width 0.25) (layer F.Cu) (net 5))
+  (segment (start 165.10762 96.60382) (end 165.1127 96.6089) (width 0.25) (layer F.Cu) (net 4))
+  (segment (start 165.10762 93.27134) (end 165.10762 96.60382) (width 0.25) (layer F.Cu) (net 4))
+  (segment (start 169.27576 96.2025) (end 167.15486 94.0816) (width 0.25) (layer F.Cu) (net 5))
+  (segment (start 167.15486 92.81858) (end 165.10762 90.77134) (width 0.25) (layer F.Cu) (net 5))
+  (segment (start 167.15486 94.0816) (end 167.15486 92.81858) (width 0.25) (layer F.Cu) (net 5))
   (segment (start 153.26614 88.11006) (end 153.29916 88.14308) (width 0.25) (layer F.Cu) (net 6))
   (segment (start 153.26614 84.86394) (end 153.26614 88.11006) (width 0.25) (layer F.Cu) (net 6))
@@
   (segment (start 145.64614 88.11006) (end 145.67916 88.14308) (width 0.25) (layer F.Cu) (net 9))
   (segment (start 145.64614 84.86394) (end 145.64614 88.11006) (width 0.25) (layer F.Cu) (net 9))
-  (segment (start 164.56553 96.67494) (end 163.82131 97.41916) (width 0.25) (layer B.Cu) (net 9))
-  (segment (start 165.6969 96.67494) (end 164.56553 96.67494) (width 0.25) (layer B.Cu) (net 9))
-  (segment (start 142.49908 97.41916) (end 140.60678 99.31146) (width 0.25) (layer B.Cu) (net 9))
-  (segment (start 163.82131 97.41916) (end 142.49908 97.41916) (width 0.25) (layer B.Cu) (net 9))
   (segment (start 140.60678 95.7707) (end 140.59916 95.76308) (width 0.25) (layer F.Cu) (net 9))
   (segment (start 140.60678 99.31146) (end 140.60678 95.7707) (width 0.25) (layer F.Cu) (net 9))
+  (segment (start 163.9697 97.41916) (end 165.1508 98.60026) (width 0.25) (layer B.Cu) (net 9))
+  (segment (start 140.60678 99.31146) (end 142.49908 97.41916) (width 0.25) (layer B.Cu) (net 9))
+  (segment (start 142.49908 97.41916) (end 163.9697 97.41916) (width 0.25) (layer B.Cu) (net 9))
   (segment (start 135.48614 88.11006) (end 135.51916 88.14308) (width 0.25) (layer F.Cu) (net 10))
   (segment (start 135.48614 84.86394) (end 135.48614 88.11006) (width 0.25) (layer F.Cu) (net 10))
@@
   (segment (start 127.86614 88.11006) (end 127.89916 88.14308) (width 0.25) (layer F.Cu) (net 13))
   (segment (start 127.86614 84.86394) (end 127.86614 88.11006) (width 0.25) (layer F.Cu) (net 13))
-  (segment (start 169.147121 90.384261) (end 169.99712 91.23426) (width 0.25) (layer B.Cu) (net 14))
-  (segment (start 168.04386 89.281) (end 169.147121 90.384261) (width 0.25) (layer B.Cu) (net 14))
-  (segment (start 159.51708 89.281) (end 168.04386 89.281) (width 0.25) (layer B.Cu) (net 14))
   (segment (start 158.37916 88.14308) (end 159.51708 89.281) (width 0.25) (layer B.Cu) (net 14))
-  (segment (start 155.83916 88.14308) (end 159.83966 92.14358) (width 0.25) (layer B.Cu) (net 15))
-  (segment (start 168.36644 92.14358) (end 169.99712 93.77426) (width 0.25) (layer B.Cu) (net 15))
-  (segment (start 159.83966 92.14358) (end 168.36644 92.14358) (width 0.25) (layer B.Cu) (net 15))
+  (segment (start 167.43426 89.281) (end 169.27576 91.1225) (width 0.25) (layer B.Cu) (net 14))
+  (segment (start 159.51708 89.281) (end 167.43426 89.281) (width 0.25) (layer B.Cu) (net 14))
+  (segment (start 155.83916 88.14308) (end 159.6517 91.95562) (width 0.25) (layer B.Cu) (net 15))
+  (segment (start 167.56888 91.95562) (end 169.27576 93.6625) (width 0.25) (layer B.Cu) (net 15))
+  (segment (start 159.6517 91.95562) (end 167.56888 91.95562) (width 0.25) (layer B.Cu) (net 15))
   (segment (start 127.90678 95.7707) (end 127.89916 95.76308) (width 0.25) (layer F.Cu) (net 16))
   (segment (start 127.90678 99.31146) (end 127.90678 95.7707) (width 0.25) (layer F.Cu) (net 16))
