File: minimal-atmega328p.sch (KiCad schematic (older format))
At the start: 9 parts, among them J1 Conn_01x14_Male, J2 Conn_01x06_Male, J3 Conn_01x14_Male, U1 ATmega328P-PU, Y1 16MHz

Commit message: add diode
Parts:
- added D1: DIODE, Diode_THT:D_A-405_P2.54mm_Vertical_AnodeUp, symbol pspice:DIODE
Connections:
- net +5V: now also D1.2 (A)
- net at C3.1, R1.2, U1.1 (~RESET~/PC6): now also D1.1 (K)
Changed lines of the file:
@@
 	7950 4250 7750 4250
-Wire Wire Line
-	7450 4250 7450 3750
-Wire Wire Line
-	7450 3750 6750 3750
 Wire Wire Line
 	7750 4250 7750 3950
@@
 $EndComp
 Wire Wire Line
-	7750 3650 7750 3450
+	7750 3650 7750 3550
 $Comp
 L power:+5V #PWR01
@@
 Wire Wire Line
 	6150 4950 6150 5250
+$Comp
+L pspice:DIODE D1
+U 1 1 5EA03DE0
+P 7450 3800
+F 0 "D1" V 7404 3928 50  0000 L CNN
+F 1 "DIODE" V 7495 3928 50  0000 L CNN
+F 2 "Diode_THT:D_A-405_P2.54mm_Vertical_AnodeUp" H 7450 3800 50  0001 C CNN
+F 3 "~" H 7450 3800 50  0001 C CNN
+	1    7450 3800
+	0    -1   -1   0
+$EndComp
+Wire Wire Line
+	7450 4250 7450 4000
+Wire Wire Line
+	7450 3600 7450 3550
+Wire Wire Line
+	7450 3550 7750 3550
+Connection ~ 7750 3550
+Wire Wire Line
+	7750 3550 7750 3450
+Wire Wire Line
+	7450 4250 7200 4250
+Wire Wire Line
+	7200 4250 7200 3750
+Wire Wire Line
+	7200 3750 6750 3750
+Connection ~ 7450 4250
 $EndSCHEMATC
