File: minimal-atmega328p.sch (KiCad schematic (older format))
At the start: 9 parts, among them J1 Conn_01x14_Male, J2 Conn_01x06_Male, J3 Conn_01x14_Male, U1 ATmega328P-PU, Y1 16MHz

Commit message: update files
Parts:
- added SW1: SW_Push, Button_Switch_THT:SW_PUSH_6mm_H5mm, symbol Switch:SW_Push
Connections:
- net GND: now also SW1.1
- net at C3.1, R1.2, U1.1 (~RESET~/PC6): now also SW1.2
Other:
- moved on the sheet: J2
Changed lines of the file:
@@
 EESchema Schematic File Version 4
 LIBS:minimal-atmega328p-cache
-EELAYER 30 0
+EELAYER 29 0
 EELAYER END
 $Descr A4 11693 8268
@@
 L Connector:Conn_01x06_Male J2
 U 1 1 5E9EC1F5
-P 8400 5600
-F 0 "J2" H 8508 5981 50  0000 C CNN
-F 1 "Conn_01x06_Male" H 8508 5890 50  0000 C CNN
-F 2 "Connector_PinHeader_2.54mm:PinHeader_1x06_P2.54mm_Vertical" H 8400 5600 50  0001 C CNN
-F 3 "~" H 8400 5600 50  0001 C CNN
-	1    8400 5600
+P 10450 5850
+F 0 "J2" H 10558 6231 50  0000 C CNN
+F 1 "Conn_01x06_Male" H 10558 6140 50  0000 C CNN
+F 2 "Connector_PinHeader_2.54mm:PinHeader_1x06_P2.54mm_Vertical" H 10450 5850 50  0001 C CNN
+F 3 "~" H 10450 5850 50  0001 C CNN
+	1    10450 5850
 	-1   0    0    -1
 $EndComp
 Wire Wire Line
-	8200 5400 7850 5400
-Wire Wire Line
-	8200 5500 7700 5500
-Wire Wire Line
-	8200 5600 7700 5600
-Wire Wire Line
-	8200 5700 7700 5700
-Wire Wire Line
-	8200 5800 7700 5800
-NoConn ~ 8200 5900
-Text Label 7700 5400 0    50   ~ 0
+	10250 5650 9900 5650
+Wire Wire Line
+	10250 5750 9750 5750
+Wire Wire Line
+	10250 5850 9750 5850
+Wire Wire Line
+	10250 5950 9750 5950
+Wire Wire Line
+	10250 6050 9750 6050
+NoConn ~ 10250 6150
+Text Label 9750 5650 0    50   ~ 0
 5V
-Text Label 7700 5500 0    50   ~ 0
+Text Label 9750 5750 0    50   ~ 0
 GND
-Text Label 7700 5600 0    50   ~ 0
+Text Label 9750 5850 0    50   ~ 0
 TXD
-Text Label 7700 5700 0    50   ~ 0
+Text Label 9750 5950 0    50   ~ 0
 RXD
-Text Label 7700 5800 0    50   ~ 0
+Text Label 9750 6050 0    50   ~ 0
 DTR
 Wire Wire Line
@@
 L power:PWR_FLAG #FLG0101
 U 1 1 5EA75A55
-P 7850 5150
-F 0 "#FLG0101" H 7850 5225 50  0001 C CNN
-F 1 "PWR_FLAG" H 7850 5323 50  0000 C CNN
-F 2 "" H 7850 5150 50  0001 C CNN
-F 3 "~" H 7850 5150 50  0001 C CNN
-	1    7850 5150
-	1    0    0    -1
-$EndComp
-Wire Wire Line
-	7850 5150 7850 5400
-Connection ~ 7850 5400
+P 9900 5400
+F 0 "#FLG0101" H 9900 5475 50  0001 C CNN
+F 1 "PWR_FLAG" H 9900 5573 50  0000 C CNN
+F 2 "" H 9900 5400 50  0001 C CNN
+F 3 "~" H 9900 5400 50  0001 C CNN
+	1    9900 5400
+	1    0    0    -1
+$EndComp
+Wire Wire Line
+	9900 5400 9900 5650
+Connection ~ 9900 5650
 NoConn ~ 5550 2250
 $Comp
 L power:+5V #PWR0105
 U 1 1 5EA7C044
-P 7500 5050
-F 0 "#PWR0105" H 7500 4900 50  0001 C CNN
-F 1 "+5V" H 7515 5223 50  0000 C CNN
-F 2 "" H 7500 5050 50  0001 C CNN
-F 3 "" H 7500 5050 50  0001 C CNN
-	1    7500 5050
-	1    0    0    -1
-$EndComp
-Wire Wire Line
-	7500 5400 7850 5400
-Wire Wire Line
-	7500 5050 7500 5400
+P 9550 5300
+F 0 "#PWR0105" H 9550 5150 50  0001 C CNN
+F 1 "+5V" H 9565 5473 50  0000 C CNN
+F 2 "" H 9550 5300 50  0001 C CNN
+F 3 "" H 9550 5300 50  0001 C CNN
+	1    9550 5300
+	1    0    0    -1
+$EndComp
+Wire Wire Line
+	9550 5650 9900 5650
+Wire Wire Line
+	9550 5300 9550 5650
 $Comp
 L power:GND #PWR0106
@@
 Wire Wire Line
 	6150 4950 6150 5250
+$Comp
+L Switch:SW_Push SW1
+U 1 1 5F7690D9
+P 7750 4700
+F 0 "SW1" V 7796 4652 50  0000 R CNN
+F 1 "SW_Push" V 7705 4652 50  0000 R CNN
+F 2 "Button_Switch_THT:SW_PUSH_6mm_H5mm" H 7750 4900 50  0001 C CNN
+F 3 "~" H 7750 4900 50  0001 C CNN
+	1    7750 4700
+	0    -1   -1   0
+$EndComp
+Wire Wire Line
+	7750 4250 7750 4500
+$Comp
+L power:GND #PWR02
+U 1 1 5F776110
+P 7750 5200
+F 0 "#PWR02" H 7750 4950 50  0001 C CNN
+F 1 "GND" H 7755 5027 50  0000 C CNN
+F 2 "" H 7750 5200 50  0001 C CNN
+F 3 "" H 7750 5200 50  0001 C CNN
+	1    7750 5200
+	1    0    0    -1
+$EndComp
+Wire Wire Line
+	7750 4900 7750 5200
 $EndSCHEMATC
